File: Hardware/edge-sens-interface-circuit.kicad_sch (KiCad schematic)
At the start: 4 parts, among them Q7 BC547

Commit message: Session 13 hardware modifications
Parts:
- renumbered Q7 to Q9, R7 to R13, R8 to R14, R9 to R15
Changed lines of the file:
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@@
 		(dnp no)
 		(fields_autoplaced yes)
-		(property "Reference" "#PWR012"
+		(property "Reference" "#PWR020"
 			(at 157.48 92.71 0)
 			(effects
@@
 		(instances
 			(project "OpenVac"
+				(path "/cfb1a53c-1978-4730-a380-294525b876d3/55098150-25e9-40bf-a15b-af880a8b89c0"
+					(reference "#PWR020")
+					(unit 1)
+				)
 				(path "/cfb1a53c-1978-4730-a380-294525b876d3/8abbe261-48c3-4668-94b5-9a917ef396bb"
 					(reference "#PWR012")
@@
 				(path "/cfb1a53c-1978-4730-a380-294525b876d3/b687b0a4-cbe8-439c-a447-5ea3319f4848"
 					(reference "#PWR016")
-					(unit 1)
-				)
-				(path "/cfb1a53c-1978-4730-a380-294525b876d3/55098150-25e9-40bf-a15b-af880a8b89c0"
-					(reference "#PWR020")
 					(unit 1)
 				)
@@
 		(dnp no)
 		(fields_autoplaced yes)
-		(property "Reference" "#PWR011"
+		(property "Reference" "#PWR019"
 			(at 148.59 107.95 0)
 			(effects
@@
 		(instances
 			(project "OpenVac"
+				(path "/cfb1a53c-1978-4730-a380-294525b876d3/55098150-25e9-40bf-a15b-af880a8b89c0"
+					(reference "#PWR019")
+					(unit 1)
+				)
 				(path "/cfb1a53c-1978-4730-a380-294525b876d3/8abbe261-48c3-4668-94b5-9a917ef396bb"
 					(reference "#PWR011")
@@
 				(path "/cfb1a53c-1978-4730-a380-294525b876d3/b687b0a4-cbe8-439c-a447-5ea3319f4848"
 					(reference "#PWR015")
-					(unit 1)
-				)
-				(path "/cfb1a53c-1978-4730-a380-294525b876d3/55098150-25e9-40bf-a15b-af880a8b89c0"
-					(reference "#PWR019")
 					(unit 1)
 				)
@@
 		(on_board yes)
 		(dnp no)
-		(property "Reference" "R8"
+		(property "Reference" "R14"
 			(at 138.684 104.14 0)
 			(effects
@@
 		(instances
 			(project "OpenVac"
+				(path "/cfb1a53c-1978-4730-a380-294525b876d3/55098150-25e9-40bf-a15b-af880a8b89c0"
+					(reference "R14")
+					(unit 1)
+				)
 				(path "/cfb1a53c-1978-4730-a380-294525b876d3/8abbe261-48c3-4668-94b5-9a917ef396bb"
 					(reference "R8")
@@
 				(path "/cfb1a53c-1978-4730-a380-294525b876d3/b687b0a4-cbe8-439c-a447-5ea3319f4848"
 					(reference "R11")
-					(unit 1)
-				)
-				(path "/cfb1a53c-1978-4730-a380-294525b876d3/55098150-25e9-40bf-a15b-af880a8b89c0"
-					(reference "R14")
 					(unit 1)
 				)
@@
 		(dnp no)
 		(fields_autoplaced yes)
-		(property "Reference" "R9"
+		(property "Reference" "R15"
 			(at 153.67 86.36 90)
 			(effects
@@
 		(instances
 			(project "OpenVac"
+				(path "/cfb1a53c-1978-4730-a380-294525b876d3/55098150-25e9-40bf-a15b-af880a8b89c0"
+					(reference "R15")
+					(unit 1)
+				)
 				(path "/cfb1a53c-1978-4730-a380-294525b876d3/8abbe261-48c3-4668-94b5-9a917ef396bb"
 					(reference "R9")
@@
 				(path "/cfb1a53c-1978-4730-a380-294525b876d3/b687b0a4-cbe8-439c-a447-5ea3319f4848"
 					(reference "R12")
-					(unit 1)
-				)
-				(path "/cfb1a53c-1978-4730-a380-294525b876d3/55098150-25e9-40bf-a15b-af880a8b89c0"
-					(reference "R15")
 					(unit 1)
 				)
@@
 		(on_board yes)
 		(dnp no)
-		(property "Reference" "Q7"
+		(property "Reference" "Q9"
 			(at 133.858 82.55 0)
 			(effects
@@
 		(instances
 			(project "OpenVac"
+				(path "/cfb1a53c-1978-4730-a380-294525b876d3/55098150-25e9-40bf-a15b-af880a8b89c0"
+					(reference "Q9")
+					(unit 1)
+				)
 				(path "/cfb1a53c-1978-4730-a380-294525b876d3/8abbe261-48c3-4668-94b5-9a917ef396bb"
 					(reference "Q7")
@@
 				(path "/cfb1a53c-1978-4730-a380-294525b876d3/b687b0a4-cbe8-439c-a447-5ea3319f4848"
 					(reference "Q8")
-					(unit 1)
-				)
-				(path "/cfb1a53c-1978-4730-a380-294525b876d3/55098150-25e9-40bf-a15b-af880a8b89c0"
-					(reference "Q9")
 					(unit 1)
 				)
@@
 		(on_board yes)
 		(dnp no)
-		(property "Reference" "R7"
+		(property "Reference" "R13"
 			(at 132.08 92.202 90)
 			(effects
@@
 		(instances
 			(project "OpenVac"
+				(path "/cfb1a53c-1978-4730-a380-294525b876d3/55098150-25e9-40bf-a15b-af880a8b89c0"
+					(reference "R13")
+					(unit 1)
+				)
 				(path "/cfb1a53c-1978-4730-a380-294525b876d3/8abbe261-48c3-4668-94b5-9a917ef396bb"
 					(reference "R7")
@@
 				(path "/cfb1a53c-1978-4730-a380-294525b876d3/b687b0a4-cbe8-439c-a447-5ea3319f4848"
 					(reference "R10")
-					(unit 1)
-				)
-				(path "/cfb1a53c-1978-4730-a380-294525b876d3/55098150-25e9-40bf-a15b-af880a8b89c0"
-					(reference "R13")
 					(unit 1)
 				)
@@
 		(dnp no)
 		(fields_autoplaced yes)
-		(property "Reference" "#PWR09"
+		(property "Reference" "#PWR017"
 			(at 143.51 77.47 0)
 			(effects
@@
 		(instances
 			(project "OpenVac"
+				(path "/cfb1a53c-1978-4730-a380-294525b876d3/55098150-25e9-40bf-a15b-af880a8b89c0"
+					(reference "#PWR017")
+					(unit 1)
+				)
 				(path "/cfb1a53c-1978-4730-a380-294525b876d3/8abbe261-48c3-4668-94b5-9a917ef396bb"
 					(reference "#PWR09")
@@
 				(path "/cfb1a53c-1978-4730-a380-294525b876d3/b687b0a4-cbe8-439c-a447-5ea3319f4848"
 					(reference "#PWR013")
-					(unit 1)
-				)
-				(path "/cfb1a53c-1978-4730-a380-294525b876d3/55098150-25e9-40bf-a15b-af880a8b89c0"
-					(reference "#PWR017")
 					(unit 1)
 				)
@@
 		(dnp no)
 		(fields_autoplaced yes)
-		(property "Reference" "#PWR010"
+		(property "Reference" "#PWR018"
 			(at 143.51 105.41 0)
 			(effects
@@
 		(instances
 			(project "OpenVac"
+				(path "/cfb1a53c-1978-4730-a380-294525b876d3/55098150-25e9-40bf-a15b-af880a8b89c0"
+					(reference "#PWR018")
+					(unit 1)
+				)
 				(path "/cfb1a53c-1978-4730-a380-294525b876d3/8abbe261-48c3-4668-94b5-9a917ef396bb"
 					(reference "#PWR010")
@@
 					(unit 1)
 				)
-				(path "/cfb1a53c-1978-4730-a380-294525b876d3/55098150-25e9-40bf-a15b-af880a8b89c0"
-					(reference "#PWR018")
-					(unit 1)
-				)
