File: Hardware/ir-sens-module.kicad_sch (KiCad schematic)
At the start: 2 parts

Commit message: Session 13 hardware modifications
Parts:
- renumbered D1 to D5, D2 to D6
Changed lines of the file:
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@@
 		(dnp no)
 		(fields_autoplaced yes)
-		(property "Reference" "D2"
+		(property "Reference" "D6"
 			(at 163.83 107.0228 90)
 			(effects
@@
 		(instances
 			(project "OpenVac"
+				(path "/cfb1a53c-1978-4730-a380-294525b876d3/55098150-25e9-40bf-a15b-af880a8b89c0/88d33abb-2da1-4302-82c1-cb5321f35028"
+					(reference "D6")
+					(unit 1)
+				)
 				(path "/cfb1a53c-1978-4730-a380-294525b876d3/8abbe261-48c3-4668-94b5-9a917ef396bb/88d33abb-2da1-4302-82c1-cb5321f35028"
 					(reference "D2")
@@
 				(path "/cfb1a53c-1978-4730-a380-294525b876d3/b687b0a4-cbe8-439c-a447-5ea3319f4848/88d33abb-2da1-4302-82c1-cb5321f35028"
 					(reference "D4")
-					(unit 1)
-				)
-				(path "/cfb1a53c-1978-4730-a380-294525b876d3/55098150-25e9-40bf-a15b-af880a8b89c0/88d33abb-2da1-4302-82c1-cb5321f35028"
-					(reference "D6")
 					(unit 1)
 				)
@@
 		(dnp no)
 		(fields_autoplaced yes)
-		(property "Reference" "D1"
+		(property "Reference" "D5"
 			(at 149.86 106.8069 90)
 			(effects
@@
 		(instances
 			(project "OpenVac"
+				(path "/cfb1a53c-1978-4730-a380-294525b876d3/55098150-25e9-40bf-a15b-af880a8b89c0/88d33abb-2da1-4302-82c1-cb5321f35028"
+					(reference "D5")
+					(unit 1)
+				)
 				(path "/cfb1a53c-1978-4730-a380-294525b876d3/8abbe261-48c3-4668-94b5-9a917ef396bb/88d33abb-2da1-4302-82c1-cb5321f35028"
 					(reference "D1")
@@
 					(unit 1)
 				)
-				(path "/cfb1a53c-1978-4730-a380-294525b876d3/55098150-25e9-40bf-a15b-af880a8b89c0/88d33abb-2da1-4302-82c1-cb5321f35028"
-					(reference "D5")
-					(unit 1)
-				)
