File: Hardware/v0.1 - Movement/sweep-brushes.kicad_sch (KiCad schematic)
At the start: 6 parts, among them J1 Brush Motor 2 (right), J2 Brush Motor 1 (left), Q1 IRF540N, Q2 IRF540N

Commit message: added session 15
Connections:
- net +12V: now also J2.1 (Pin_1); no longer J2.2 (Pin_2)
- net at Q2.2 (D): now also J2.2 (Pin_2); no longer J2.1 (Pin_1)
Other:
- moved on the sheet: J1, J2, Q1, R2
Changed lines of the file:
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@@
 	)
 	(junction
-		(at 146.05 81.28)
+		(at 146.05 78.74)
 		(diameter 0)
 		(color 0 0 0 0)
@@
 	(wire
 		(pts
-			(xy 146.05 80.01) (xy 146.05 81.28)
+			(xy 146.05 77.47) (xy 146.05 78.74)
 		)
 		(stroke
@@
 	(wire
 		(pts
-			(xy 129.54 88.9) (xy 140.97 88.9)
+			(xy 146.05 107.95) (xy 146.05 109.22)
 		)
 		(stroke
@@
 	(wire
 		(pts
-			(xy 146.05 107.95) (xy 146.05 109.22)
+			(xy 129.54 86.36) (xy 140.97 86.36)
 		)
 		(stroke
@@
 	(hierarchical_label "rightBrushActivate"
 		(shape input)
-		(at 146.05 80.01 90)
+		(at 146.05 77.47 90)
 		(fields_autoplaced yes)
 		(effects
@@
 	(symbol
 		(lib_id "power:+12V")
-		(at 129.54 119.38 270)
+		(at 129.54 114.3 270)
 		(unit 1)
 		(exclude_from_sim no)
@@
 		(fields_autoplaced yes)
 		(property "Reference" "#PWR02"
-			(at 125.73 119.38 0)
+			(at 125.73 114.3 0)
 			(effects
 				(font
@@
 		)
 		(property "Value" "+12V"
-			(at 133.35 119.3799 90)
+			(at 133.35 114.2999 90)
 			(effects
 				(font
@@
 		)
 		(property "Footprint" ""
-			(at 129.54 119.38 0)
+			(at 129.54 114.3 0)
 			(effects
 				(font
@@
 		)
 		(property "Datasheet" ""
-			(at 129.54 119.38 0)
+			(at 129.54 114.3 0)
 			(effects
 				(font
@@
 		)
 		(property "Description" "Power symbol creates a global label with name \"+12V\""
-			(at 129.54 119.38 0)
+			(at 129.54 114.3 0)
 			(effects
 				(font
@@
 	(symbol
 		(lib_id "power:GND")
-		(at 153.67 81.28 90)
+		(at 153.67 78.74 90)
 		(unit 1)
 		(exclude_from_sim no)
@@
 		(fields_autoplaced yes)
 		(property "Reference" "#PWR07"
-			(at 160.02 81.28 0)
+			(at 160.02 78.74 0)
 			(effects
 				(font
@@
 		)
 		(property "Value" "GND"
-			(at 157.48 81.2799 90)
+			(at 157.48 78.7399 90)
 			(effects
 				(font
@@
 		)
 		(property "Footprint" ""
-			(at 153.67 81.28 0)
+			(at 153.67 78.74 0)
 			(effects
 				(font
@@
 		)
 		(property "Datasheet" ""
-			(at 153.67 81.28 0)
+			(at 153.67 78.74 0)
 			(effects
 				(font
@@
 		)
 		(property "Description" "Power symbol creates a global label with name \"GND\" , ground"
-			(at 153.67 81.28 0)
+			(at 153.67 78.74 0)
 			(effects
 				(font
@@
 	(symbol
 		(lib_id "power:GND")
-		(at 151.13 88.9 90)
+		(at 151.13 86.36 90)
 		(unit 1)
 		(exclude_from_sim no)
@@
 		(fields_autoplaced yes)
 		(property "Reference" "#PWR03"
-			(at 157.48 88.9 0)
+			(at 157.48 86.36 0)
 			(effects
 				(font
@@
 		)
 		(property "Value" "GND"
-			(at 154.94 88.8999 90)
+			(at 154.94 86.3599 90)
 			(effects
 				(font
@@
 		)
 		(property "Footprint" ""
-			(at 151.13 88.9 0)
+			(at 151.13 86.36 0)
 			(effects
 				(font
@@
 		)
 		(property "Datasheet" ""
-			(at 151.13 88.9 0)
+			(at 151.13 86.36 0)
 			(effects
 				(font
@@
 		)
 		(property "Description" "Power symbol creates a global label with name \"GND\" , ground"
-			(at 151.13 88.9 0)
+			(at 151.13 86.36 0)
 			(effects
 				(font
@@
 	(symbol
 		(lib_id "Connector:Conn_01x02_Pin")
-		(at 124.46 88.9 0)
+		(at 124.46 86.36 0)
 		(unit 1)
 		(exclude_from_sim no)
@@
 		(fields_autoplaced yes)
 		(property "Reference" "J1"
+			(at 125.095 81.28 0)
+			(effects
+				(font
+					(size 1.27 1.27)
+				)
+			)
+		)
+		(property "Value" "Brush Motor 2 (right)"
 			(at 125.095 83.82 0)
 			(effects
@@
 			)
 		)
-		(property "Value" "Brush Motor 2 (right)"
-			(at 125.095 86.36 0)
-			(effects
-				(font
-					(size 1.27 1.27)
-				)
-			)
-		)
 		(property "Footprint" "Connector_JST:JST_PH_B2B-PH-K_1x02_P2.00mm_Vertical"
-			(at 124.46 88.9 0)
+			(at 124.46 86.36 0)
 			(effects
 				(font
@@
 		)
 		(property "Datasheet" "~"
-			(at 124.46 88.9 0)
+			(at 124.46 86.36 0)
 			(effects
 				(font
@@
 		)
 		(property "Description" "Generic connector, single row, 01x02, script generated"
-			(at 124.46 88.9 0)
+			(at 124.46 86.36 0)
 			(effects
 				(font
@@
 	(symbol
 		(lib_id "Connector:Conn_01x02_Pin")
-		(at 124.46 116.84 0)
+		(at 124.46 114.3 0)
 		(unit 1)
 		(exclude_from_sim no)
@@
 		(fields_autoplaced yes)
 		(property "Reference" "J2"
+			(at 125.095 109.22 0)
+			(effects
+				(font
+					(size 1.27 1.27)
+				)
+			)
+		)
+		(property "Value" "Brush Motor 1 (left)"
 			(at 125.095 111.76 0)
 			(effects
@@
 			)
 		)
-		(property "Value" "Brush Motor 1 (left)"
-			(at 125.095 114.3 0)
-			(effects
-				(font
-					(size 1.27 1.27)
-				)
-			)
-		)
 		(property "Footprint" "Connector_JST:JST_PH_B2B-PH-K_1x02_P2.00mm_Vertical"
-			(at 124.46 116.84 0)
+			(at 124.46 114.3 0)
 			(effects
 				(font
@@
 		)
 		(property "Datasheet" "~"
-			(at 124.46 116.84 0)
+			(at 124.46 114.3 0)
 			(effects
 				(font
@@
 		)
 		(property "Description" "Generic connector, single row, 01x02, script generated"
-			(at 124.46 116.84 0)
+			(at 124.46 114.3 0)
 			(effects
 				(font
@@
 	(symbol
 		(lib_id "power:+12V")
-		(at 129.54 91.44 270)
+		(at 129.54 88.9 270)
 		(unit 1)
 		(exclude_from_sim no)
@@
 		(fields_autoplaced yes)
 		(property "Reference" "#PWR01"
-			(at 125.73 91.44 0)
+			(at 125.73 88.9 0)
 			(effects
 				(font
@@
 		)
 		(property "Value" "+12V"
-			(at 133.35 91.4399 90)
+			(at 133.35 88.8999 90)
 			(effects
 				(font
@@
 		)
 		(property "Footprint" ""
-			(at 129.54 91.44 0)
+			(at 129.54 88.9 0)
 			(effects
 				(font
@@
 		)
 		(property "Datasheet" ""
-			(at 129.54 91.44 0)
+			(at 129.54 88.9 0)
 			(effects
 				(font
@@
 		)
 		(property "Description" "Power symbol creates a global label with name \"+12V\""
-			(at 129.54 91.44 0)
+			(at 129.54 88.9 0)
 			(effects
 				(font
@@
 	(symbol
 		(lib_id "Device:R")
-		(at 149.86 81.28 90)
+		(at 149.86 78.74 90)
 		(unit 1)
 		(exclude_from_sim no)
@@
 		(fields_autoplaced yes)
 		(property "Reference" "R2"
+			(at 149.86 72.39 90)
+			(effects
+				(font
+					(size 1.27 1.27)
+				)
+			)
+		)
+		(property "Value" "10k"
 			(at 149.86 74.93 90)
 			(effects
@@
 			)
 		)
-		(property "Value" "10k"
-			(at 149.86 77.47 90)
-			(effects
-				(font
-					(size 1.27 1.27)
-				)
-			)
-		)
 		(property "Footprint" "Resistor_THT:R_Axial_DIN0207_L6.3mm_D2.5mm_P10.16mm_Horizontal"
-			(at 149.86 83.058 90)
+			(at 149.86 80.518 90)
 			(effects
 				(font
@@
 		)
 		(property "Datasheet" "~"
-			(at 149.86 81.28 0)
+			(at 149.86 78.74 0)
 			(effects
 				(font
@@
 		)
 		(property "Description" "Resistor"
-			(at 149.86 81.28 0)
+			(at 149.86 78.74 0)
 			(effects
 				(font
@@
 	(symbol
 		(lib_id "Transistor_FET:IRF540N")
-		(at 146.05 86.36 90)
+		(at 146.05 83.82 90)
 		(mirror x)
 		(unit 1)
@@
 		(dnp no)
 		(property "Reference" "Q1"
+			(at 146.05 90.17 90)
+			(effects
+				(font
+					(size 1.27 1.27)
+				)
+			)
+		)
+		(property "Value" "IRF540N"
 			(at 146.05 92.71 90)
 			(effects
@@
 			)
 		)
-		(property "Value" "IRF540N"
-			(at 146.05 95.25 90)
-			(effects
-				(font
-					(size 1.27 1.27)
-				)
-			)
-		)
 		(property "Footprint" "Package_TO_SOT_THT:TO-220-3_Vertical"
-			(at 147.955 91.44 0)
+			(at 147.955 88.9 0)
 			(effects
 				(font
@@
 		)
 		(property "Datasheet" "http://www.irf.com/product-info/datasheets/data/irf540n.pdf"
-			(at 149.86 91.44 0)
+			(at 149.86 88.9 0)
 			(effects
 				(font
@@
 		)
 		(property "Description" "33A Id, 100V Vds, HEXFET N-Channel MOSFET, TO-220"
-			(at 146.05 86.36 0)
-			(effects
-				(font
+			(at 146.05 83.82 0)
+			(effects
+				(font
