File: Hardware/v0.1 - Movement/openVac-v0.1.kicad_sch (KiCad schematic)
At the start: 0 parts

Commit message: added session 15
Parts:
- added H1: 12V (external in), MountingHole:MountingHole_2.2mm_M2_DIN965_Pad, symbol Mechanical:MountingHole_Pad
- added H2: GND (external in), MountingHole:MountingHole_2.2mm_M2_DIN965_Pad, symbol Mechanical:MountingHole_Pad
- added J3: Brush Header, Connector_JST:JST_PH_B3B-PH-K_1x03_P2.00mm_Vertical, symbol Connector:Conn_01x03_Pin
- added J6: Vacuum Header, Connector_JST:JST_PH_B2B-PH-K_1x02_P2.00mm_Vertical, symbol Connector:Conn_01x02_Pin
Connections:
- net Main Brush/mainBrushActivate: now also J3.1 (Pin_1)
- net Sweep Brushes/leftBrushActivate: now also J3.2 (Pin_2)
- net Sweep Brushes/rightBrushActivate: now also J3.3 (Pin_3)
- new net +12V: H1.1
- new net GND: H2.1
- new net Vacuum Turbine/PWM: J6.2 (Pin_2)
- new net Vacuum Turbine/Tach: J6.1 (Pin_1)
Other:
- added sheet Vacuum Turbine (vacuum.kicad_sch)

Commit message: Github Desktop Backup
Parts:
- added J9: Motor Header, Connector_JST:JST_PH_B6B-PH-K_1x06_P2.00mm_Vertical, symbol Connector:Conn_01x06_Pin
Connections:
- new net Motors/(left) forwardActive: J9.5 (Pin_5)
- new net Motors/(left) reverseActive: J9.6 (Pin_6)
- new net Motors/(left) sense^{analog}: J9.4 (Pin_4)
- new net Motors/(right) forwardActive: J9.2 (Pin_2)
- new net Motors/(right) reverseActive: J9.3 (Pin_3)
- new net Motors/(right) sense^{analog}: J9.1 (Pin_1)
Other:
- added sheet Motors (untitled.kicad_sch)

Commit message: added session 17
Parts:
- added H3: 5V (external in), MountingHole:MountingHole_2.2mm_M2_DIN965_Pad, symbol Mechanical:MountingHole_Pad
- added H4: 3.3V (external in), MountingHole:MountingHole_2.2mm_M2_DIN965_Pad, symbol Mechanical:MountingHole_Pad
- J3: value Brush Header -> Brush Header (control)
- J6: value Vacuum Header -> Vacuum Header (control)
- J9: value Motor Header -> Motor Header (control)
Connections:
- new net +3.3V: H4.1
- new net +5V: H3.1
Other:
- company: (none) -> Karl Wünsche
- title: (none) -> v0.1 Movement Development Board
- moved on the sheet: J3, J6, J9
