File: Hardware/v0.1 - Movement/vacuum.kicad_sch (KiCad schematic)
At the start: 1 part, among them J5 Vacuum

Commit message: Github Desktop Backup
Changed lines of the file:
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@@
 	)
 	(hierarchical_label "Tach"
-		(shape input)
+		(shape output)
 		(at 143.51 92.71 0)
 		(fields_autoplaced yes)

Commit message: added session 17
Other:
- company: (none) -> Karl Wünsche
- title: (none) -> Vacuum Connector
- moved on the sheet: J5
Changed lines of the file:
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@@
 	(paper "A4")
 	(title_block
+		(title "Vacuum Connector")
+		(date "2024-07-20")
 		(rev "v0.1")
+		(company "Karl Wünsche")
 	)
 	(hierarchical_label "Tach"
 		(shape output)
-		(at 143.51 92.71 0)
+		(at 146.05 101.6 0)
 		(fields_autoplaced yes)
 		(effects
@@
 	(hierarchical_label "PWM"
 		(shape input)
-		(at 143.51 90.17 0)
+		(at 146.05 99.06 0)
 		(fields_autoplaced yes)
 		(effects
@@
 	(symbol
 		(lib_id "power:+12V")
-		(at 143.51 85.09 270)
+		(at 146.05 93.98 270)
 		(unit 1)
 		(exclude_from_sim no)
@@
 		(fields_autoplaced yes)
 		(property "Reference" "#PWR012"
-			(at 139.7 85.09 0)
+			(at 142.24 93.98 0)
 			(effects
 				(font
@@
 		)
 		(property "Value" "+12V"
-			(at 147.32 85.0899 90)
+			(at 149.86 93.9799 90)
 			(effects
 				(font
@@
 		)
 		(property "Footprint" ""
-			(at 143.51 85.09 0)
+			(at 146.05 93.98 0)
 			(effects
 				(font
@@
 		)
 		(property "Datasheet" ""
-			(at 143.51 85.09 0)
+			(at 146.05 93.98 0)
 			(effects
 				(font
@@
 		)
 		(property "Description" "Power symbol creates a global label with name \"+12V\""
-			(at 143.51 85.09 0)
+			(at 146.05 93.98 0)
 			(effects
 				(font
@@
 	(symbol
 		(lib_id "power:GND")
-		(at 143.51 87.63 90)
+		(at 146.05 96.52 90)
 		(unit 1)
 		(exclude_from_sim no)
@@
 		(fields_autoplaced yes)
 		(property "Reference" "#PWR013"
-			(at 149.86 87.63 0)
+			(at 152.4 96.52 0)
 			(effects
 				(font
@@
 		)
 		(property "Value" "GND"
-			(at 147.32 87.6299 90)
+			(at 149.86 96.5199 90)
 			(effects
 				(font
@@
 		)
 		(property "Footprint" ""
-			(at 143.51 87.63 0)
+			(at 146.05 96.52 0)
 			(effects
 				(font
@@
 		)
 		(property "Datasheet" ""
-			(at 143.51 87.63 0)
+			(at 146.05 96.52 0)
 			(effects
 				(font
@@
 		)
 		(property "Description" "Power symbol creates a global label with name \"GND\" , ground"
-			(at 143.51 87.63 0)
+			(at 146.05 96.52 0)
 			(effects
 				(font
@@
 	(symbol
 		(lib_id "Connector:Conn_01x04_Pin")
-		(at 138.43 87.63 0)
+		(at 140.97 96.52 0)
 		(unit 1)
 		(exclude_from_sim no)
@@
 		(fields_autoplaced yes)
 		(property "Reference" "J5"
-			(at 139.065 80.01 0)
+			(at 141.605 88.9 0)
 			(effects
 				(font
@@
 		)
 		(property "Value" "Vacuum"
-			(at 139.065 82.55 0)
+			(at 141.605 91.44 0)
 			(effects
 				(font
@@
 		)
 		(property "Footprint" "Connector_JST:JST_PH_B4B-PH-K_1x04_P2.00mm_Vertical"
-			(at 138.43 87.63 0)
+			(at 140.97 96.52 0)
 			(effects
 				(font
@@
 		)
 		(property "Datasheet" "~"
-			(at 138.43 87.63 0)
+			(at 140.97 96.52 0)
 			(effects
 				(font
@@
 		)
 		(property "Description" "Generic connector, single row, 01x04, script generated"
-			(at 138.43 87.63 0)
-			(effects
-				(font
+			(at 140.97 96.52 0)
+			(effects
+				(font
