File: Hardware/v0.1 - Movement/openVac-v0.1.kicad_pcb (KiCad board)
At the start: 2 copper layers, 167 x 100 mm, 9 parts, among them J1 Brush Motor 2 (right), J2 Brush Motor 1 (left), J4 Brush Motor Main, Q1 IRF540N, Q2 IRF540N, Q4 IRF540N

Commit message: added session 15
Parts:
- added H1: 12V (external in), MountingHole:MountingHole_2.2mm_M2_DIN965_Pad, F.Cu at (116.6, 146.0)
- added H2: GND (external in), MountingHole:MountingHole_2.2mm_M2_DIN965_Pad, F.Cu at (123.8, 146.0)
- added J3: Brush Header, Connector_JST:JST_PH_B3B-PH-K_1x03_P2.00mm_Vertical, F.Cu at (136.6, 145.4)
- added J5: Vacuum, Connector_JST:JST_PH_B4B-PH-K_1x04_P2.00mm_Vertical, F.Cu at (175.6, 146.6)
- added J6: Vacuum Header, Connector_JST:JST_PH_B2B-PH-K_1x02_P2.00mm_Vertical, F.Cu at (149.6, 146.6)
- moved J4 12.6 mm to (194.6, 146.6)
- moved Q4 12.6 mm to (196.1, 135.0)
- moved R3 12.6 mm to (198.6, 128.0)
- moved J1 9.66 mm to (226.1, 104.5)
- moved J2 9.66 mm to (77.5, 106.3)
- moved Q1 9.66 mm to (214.5, 102.9)
- moved Q2 9.66 mm to (89.0, 107.9)
- moved R1 9.66 mm to (96.0, 110.5)
- moved R2 9.66 mm to (207.5, 100.3)
Connections:
- J2 pad 1: Net-(J2-Pin_1) -> +12V
- J2 pad 2: +12V -> Net-(J2-Pin_2)
- Q2 pad 2: Net-(J2-Pin_1) -> Net-(J2-Pin_2)
Other:
- board text added: "+12V"
- board text added: "GND"
- board text added: "PWM"
- board text added: "Tach"
- board text added: "left brush"
- board text added: "main brush"
- board text added: "right brush"

Commit message: Github Desktop Backup
Parts:
- removed H1: 12V (external in), MountingHole:MountingHole_2.2mm_M2_DIN965_Pad
- removed H2: GND (external in), MountingHole:MountingHole_2.2mm_M2_DIN965_Pad
- removed J1: Brush Motor 2 (right), Connector_JST:JST_PH_B2B-PH-K_1x02_P2.00mm_Vertical
- removed J2: Brush Motor 1 (left), Connector_JST:JST_PH_B2B-PH-K_1x02_P2.00mm_Vertical
- removed J3: Brush Header, Connector_JST:JST_PH_B3B-PH-K_1x03_P2.00mm_Vertical
- removed J4: Brush Motor Main, Connector_JST:JST_PH_B2B-PH-K_1x02_P2.00mm_Vertical
- removed J5: Vacuum, Connector_JST:JST_PH_B4B-PH-K_1x04_P2.00mm_Vertical
- removed J6: Vacuum Header, Connector_JST:JST_PH_B2B-PH-K_1x02_P2.00mm_Vertical
- removed Q1, Q2, Q4: IRF540N, Package_TO_SOT_THT:TO-220-3_Vertical
- removed R1, R2, R3: 10k, Resistor_THT:R_Axial_DIN0207_L6.3mm_D2.5mm_P10.16mm_Horizontal
Other:
- board size 167 x 100 mm -> 171.5 x 100 mm
- board text removed: "+12V"
- board text removed: "GND"
- board text removed: "PWM"
- board text removed: "Tach"
- board text removed: "left brush"
- board text removed: "main brush"
- board text removed: "right brush"

Commit message: added session 17
Parts:
- added C1: 0.1uF, Capacitor_THT:CP_Radial_D4.0mm_P1.50mm, F.Cu at (140.5, 99.2)
- added C2: 0.1uF, Capacitor_THT:CP_Radial_D4.0mm_P1.50mm, F.Cu at (140.5, 104.8)
- added H1: 12V (external in), MountingHole:MountingHole_2.2mm_M2_DIN965_Pad, F.Cu at (161.8, 75.3)
- added H2: GND (external in), MountingHole:MountingHole_2.2mm_M2_DIN965_Pad, F.Cu at (161.8, 80.6)
- added H3: 5V (external in), MountingHole:MountingHole_2.2mm_M2_DIN965_Pad, F.Cu at (161.8, 86.0)
- added H4: 3.3V (external in), MountingHole:MountingHole_2.2mm_M2_DIN965_Pad, F.Cu at (161.8, 91.3)
- added J1: Brush Motor 2 (right), Connector_JST:JST_PH_B2B-PH-K_1x02_P2.00mm_Vertical, F.Cu at (225.6, 98.0)
- added J2: Brush Motor 1 (left), Connector_JST:JST_PH_B2B-PH-K_1x02_P2.00mm_Vertical, F.Cu at (66.5, 100.0)
- added J3: Brush Header (control), Connector_JST:JST_PH_B3B-PH-K_1x03_P2.00mm_Vertical, F.Cu at (116.5, 148.0)
- added J4: Brush Motor Main, Connector_JST:JST_PH_B2B-PH-K_1x02_P2.00mm_Vertical, F.Cu at (181.6, 149.1)
- added J5: Vacuum, Connector_JST:JST_PH_B4B-PH-K_1x04_P2.00mm_Vertical, F.Cu at (163.6, 148.0)
- added J6: Vacuum Header (control), Connector_JST:JST_PH_B2B-PH-K_1x02_P2.00mm_Vertical, F.Cu at (130.6, 148.0)
- added J7: Motor (left), Connector_JST:JST_PH_B6B-PH-K_1x06_P2.00mm_Vertical, F.Cu at (67.5, 120.5)
- added J8: Motor (right), Connector_JST:JST_PH_B6B-PH-K_1x06_P2.00mm_Vertical, F.Cu at (225.6, 120.5)
- added J9: Motor Header (control), Connector_JST:JST_PH_B6B-PH-K_1x06_P2.00mm_Vertical, F.Cu at (96.5, 148.0)
- added Q1: IRF540N, Package_TO_SOT_THT:TO-220-3_Vertical, F.Cu at (217.0, 100.6)
- added Q10: IRF540N, Package_TO_SOT_THT:TO-220-3_Vertical, F.Cu at (137.2, 88.5)
- added Q11: IRF9540N, Package_TO_SOT_THT:TO-220-3_Vertical, F.Cu at (137.2, 94.4)
- added Q12: IRF540N, Package_TO_SOT_THT:TO-220-3_Vertical, F.Cu at (148.8, 76.5)
- added Q13: IRF540N, Package_TO_SOT_THT:TO-220-3_Vertical, F.Cu at (148.8, 82.5)
- added Q14: IRF9540N, Package_TO_SOT_THT:TO-220-3_Vertical, F.Cu at (148.8, 88.5)
- added Q15: IRF540N, Package_TO_SOT_THT:TO-220-3_Vertical, F.Cu at (148.8, 94.4)
- added Q2: IRF540N, Package_TO_SOT_THT:TO-220-3_Vertical, F.Cu at (75.0, 95.4)
- added Q3: IRF540N, Package_TO_SOT_THT:TO-220-3_Vertical, F.Cu at (125.7, 76.5)
- added Q4: IRF540N, Package_TO_SOT_THT:TO-220-3_Vertical, F.Cu at (179.0, 140.0)
- added Q5: IRF9540N, Package_TO_SOT_THT:TO-220-3_Vertical, F.Cu at (125.7, 82.5)
- added Q6: IRF540N, Package_TO_SOT_THT:TO-220-3_Vertical, F.Cu at (125.7, 88.5)
- added Q7: IRF540N, Package_TO_SOT_THT:TO-220-3_Vertical, F.Cu at (125.7, 94.4)
- added Q8: IRF9540N, Package_TO_SOT_THT:TO-220-3_Vertical, F.Cu at (137.2, 76.5)
- added Q9: IRF540N, Package_TO_SOT_THT:TO-220-3_Vertical, F.Cu at (137.2, 82.5)
- added R1: 10k, Resistor_THT:R_Axial_DIN0207_L6.3mm_D2.5mm_P10.16mm_Horizontal, F.Cu at (83.5, 92.9)
- added R10: 10K, Resistor_THT:R_Axial_DIN0207_L6.3mm_D2.5mm_P10.16mm_Horizontal, F.Cu at (110.7, 98.9)
- added R11: 10, Resistor_THT:R_Axial_DIN0207_L6.3mm_D2.5mm_P10.16mm_Horizontal, F.Cu at (110.7, 103.0)
- added R12: 10K, Resistor_THT:R_Axial_DIN0207_L6.3mm_D2.5mm_P10.16mm_Horizontal, F.Cu at (110.7, 107.0)
- added R13: 10K, Resistor_THT:R_Axial_DIN0207_L6.3mm_D2.5mm_P10.16mm_Horizontal, F.Cu at (110.7, 111.1)
- added R14: 10k, Resistor_THT:R_Axial_DIN0207_L6.3mm_D2.5mm_P10.16mm_Horizontal, F.Cu at (110.7, 115.1)
- added R15: 10, Resistor_THT:R_Axial_DIN0207_L6.3mm_D2.5mm_P10.16mm_Horizontal, F.Cu at (110.7, 119.2)
- added R16: 5.1k, Resistor_THT:R_Axial_DIN0207_L6.3mm_D2.5mm_P10.16mm_Horizontal, F.Cu at (110.7, 123.2)
- added R17: 10k, Resistor_THT:R_Axial_DIN0207_L6.3mm_D2.5mm_P10.16mm_Horizontal, F.Cu at (110.7, 127.3)
- added R18: 10K, Resistor_THT:R_Axial_DIN0207_L6.3mm_D2.5mm_P10.16mm_Horizontal, F.Cu at (110.7, 131.3)
- added R19: 10K, Resistor_THT:R_Axial_DIN0207_L6.3mm_D2.5mm_P10.16mm_Horizontal, F.Cu at (110.7, 135.4)
- added R2: 10k, Resistor_THT:R_Axial_DIN0207_L6.3mm_D2.5mm_P10.16mm_Horizontal, F.Cu at (208.6, 103.1)
- added R3: 10k, Resistor_THT:R_Axial_DIN0207_L6.3mm_D2.5mm_P10.16mm_Horizontal, F.Cu at (176.4, 131.5)
- added R4: 5.1k, Resistor_THT:R_Axial_DIN0207_L6.3mm_D2.5mm_P10.16mm_Horizontal, F.Cu at (110.7, 74.6)
- added R5: 10K, Resistor_THT:R_Axial_DIN0207_L6.3mm_D2.5mm_P10.16mm_Horizontal, F.Cu at (110.7, 78.7)
- added R6: 10K, Resistor_THT:R_Axial_DIN0207_L6.3mm_D2.5mm_P10.16mm_Horizontal, F.Cu at (110.7, 82.7)
- added R7: 10k, Resistor_THT:R_Axial_DIN0207_L6.3mm_D2.5mm_P10.16mm_Horizontal, F.Cu at (110.7, 86.8)
- added R8: 10k, Resistor_THT:R_Axial_DIN0207_L6.3mm_D2.5mm_P10.16mm_Horizontal, F.Cu at (110.7, 90.8)
- added R9: 10K, Resistor_THT:R_Axial_DIN0207_L6.3mm_D2.5mm_P10.16mm_Horizontal, F.Cu at (110.7, 94.9)
Routing:
- net /Vacuum Turbine/Tach: track 0.00 -> 41.5 mm
- net /Vacuum Turbine/PWM: track 0.00 -> 36.7 mm
- net /Sweep Brushes/leftBrushActivate: track 0.00 -> 9.55 mm
- net /Main Brush/mainBrushActivate: track 0.00 -> 9.55 mm
- net /Sweep Brushes/rightBrushActivate: track 0.00 -> 9.50 mm
- net Net-(J4-Pin_1): track 0.00 -> 9.12 mm
- net Net-(J1-Pin_1): track 0.00 -> 8.56 mm
- net Net-(J2-Pin_2): track 0.00 -> 8.53 mm

Commit message: added session 18
Parts:
- moved H1 115.8 mm to (72.0, 148.5), turned to 90 degrees
- moved H2 111.9 mm to (67.5, 141.0), turned to 90 degrees
- moved R16 108.5 mm to (219.1, 126.5), turned to 180 degrees
- moved R15 108.4 mm to (219.1, 120.5), turned to 180 degrees
- moved H3 102.9 mm to (80.0, 148.5), turned to 90 degrees
- moved H4 93.3 mm to (88.0, 148.5), turned to 90 degrees
- moved R19 92.5 mm to (196.2, 100.1), turned to 180 degrees
- moved C2 78.8 mm to (214.8, 131.0), turned to 180 degrees
- moved R18 77.9 mm to (186.0, 111.6)
- moved R17 75.4 mm to (186.0, 123.5)
- moved C1 70.7 mm to (77.3, 131.0)
- moved R14 70.5 mm to (180.7, 123.5), turned to 180 degrees
- moved R13 70.0 mm to (180.7, 111.6), turned to 180 degrees
- moved R4 64.1 mm to (73.0, 126.5)
- moved R12 60.2 mm to (170.5, 100.1)
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Routing:
- net /Vacuum Turbine/Tach: track 41.5 -> 0.00 mm
- net /Vacuum Turbine/PWM: track 36.7 -> 0.00 mm
- net Net-(Q3-D): track 0.00 -> 27.9 mm
- net /Motors/(left) reverseActive: track 0.00 -> 26.0 mm
- net /Motors/(left) forwardActive: track 0.00 -> 19.9 mm
- net Net-(J7-Pin_6): track 0.00 -> 12.8 mm
- net Net-(Q8-G): track 0.00 -> 12.2 mm
- net /Motors/(left) sense^{analog}: track 0.00 -> 11.7 mm
- net /Sweep Brushes/leftBrushActivate: track 9.55 -> 0.00 mm
- net /Main Brush/mainBrushActivate: track 9.55 -> 0.00 mm
- net /Sweep Brushes/rightBrushActivate: track 9.50 -> 0.00 mm
- net Net-(J4-Pin_1): track 9.12 -> 0.00 mm
- net Net-(J1-Pin_1): track 8.56 -> 0.00 mm
- net Net-(J2-Pin_2): track 8.53 -> 0.00 mm
- net Net-(J7-Pin_1): track 0.00 -> 5.42 mm
- added copper zone on F.Cu, net GND

Commit message: added session 19
Parts:
- moved R17 23.4 mm to (186.0, 100.1)
- moved Q13 12.0 mm to (188.6, 106.5)
- moved Q15 12.0 mm to (188.6, 118.5)
- moved R18 11.9 mm to (186.0, 123.5)
- moved R19 11.5 mm to (196.2, 111.6)
- moved H2 4.50 mm to (72.0, 141.0)
Routing:
- net +12V: track 0.00 -> 322.5 mm
- net +5V: track 0.00 -> 189.6 mm
- net +3.3V: track 0.00 -> 162.6 mm
- net /Motors/(right) sense^{analog}: track 0.00 -> 142.3 mm
- net /Motors/(right) forwardActive: track 0.00 -> 127.0 mm
- net /Sweep Brushes/rightBrushActivate: track 0.00 -> 118.6 mm, vias 0 -> 1
- net /Motors/(right) reverseActive: track 0.00 -> 114.6 mm
- net /Sweep Brushes/leftBrushActivate: track 0.00 -> 90.9 mm
- net Net-(J7-Pin_5): track 0.00 -> 76.3 mm
- net /Main Brush/mainBrushActivate: track 0.00 -> 71.9 mm
- net Net-(J8-Pin_5): track 0.00 -> 68.6 mm
- net Net-(J8-Pin_6): track 0.00 -> 65.5 mm
- net /Motors/(left) sense^{analog}: track 11.7 -> 63.1 mm
- net /Motors/(left) forwardActive: track 19.9 -> 65.4 mm
- net /Vacuum Turbine/Tach: track 0.00 -> 40.8 mm
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- added copper zone on B.Cu, net GND
Other:
- board text added: "12V GND"
- board text added: "12V GND PT+ PT- IR- IR+"
- board text added: "12V GND PWM Tach"
- board text added: "Control"
- board text added: "GND 12V"
- board text added: "IR+ IR- PT- PT+ GND 12V"
- board text added: "Power"
